File: EdgeBerry.kicad_pcb (KiCad board)
At the start: 2 copper layers, 135 x 90 mm, 161 parts, among them P1 12Vin, Q1 BC547, Q2 BC547, Q3 BC547, SW1 SW_PUSH, U1 24LC256, U2 LM2596

Commit message: Schematic: cleanup + increased readability
Parts:
- C1: value 680uF -> 220uF
- U2: value LM2596 -> LM2596S-5.0
Connections:
- net status1_green renamed LED_green
- net status1_red renamed LED_red
